File: main.brd (EAGLE design)
At the start: 76.2 x 36.4 mm, 7 parts

Commit message: milestone, reroute
Connections:
- net AUDIO_L: now also GENERAL_XPN.7; no longer GENERAL_XPN.5
- net AUDIO_R: now also GENERAL_XPN.9; no longer GENERAL_XPN.6
- net GND: now also GENERAL_XPN.5; no longer GENERAL_XPN.2
- net SPI_CLK: now also GENERAL_XPN.2; no longer GENERAL_XPN.8
- net SPI_CS: now also GENERAL_XPN.8; no longer GENERAL_XPN.7
- net SPI_MISO: now also GENERAL_XPN.6; no longer GENERAL_XPN.10
- net SPI_MOSI: now also GENERAL_XPN.4; no longer GENERAL_XPN.9
Routing:
- net +3V3: track 0.00 -> 96.3 mm
- net ROTENC3_B: track 0.00 -> 81.0 mm
- net ROTENC4_A: track 0.00 -> 79.0 mm, vias 0 -> 1
- net AUDIO_L: track 0.00 -> 76.9 mm
- net AUDIO_R: track 0.00 -> 65.8 mm
- net ROTENC4_B: track 0.00 -> 58.1 mm, vias 0 -> 3
- net +5V: track 0.00 -> 57.1 mm, vias 0 -> 1
- net ROTENC2_A: track 0.00 -> 54.6 mm, vias 0 -> 1
- net ROTENC3_A: track 0.00 -> 52.9 mm, vias 0 -> 2
- net ROTENC1_B: track 0.00 -> 50.6 mm, vias 0 -> 1
- net ROTENC2_B: track 0.00 -> 48.3 mm, vias 0 -> 3
- net SCR_BL: track 0.00 -> 45.9 mm, vias 0 -> 1
- net +12V: track 0.00 -> 43.4 mm
- net SCR_DC: track 0.00 -> 42.9 mm, vias 0 -> 2
- net ROTENC1_A: track 0.00 -> 42.6 mm
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Other:
- board size 76.2 x 36.4 mm -> 76.2 x 37.6 mm

Commit message: Added 8 channel audio xpn to general board (inc. pdf)
Parts:
- removed AUDIO_MAIN: (no value), pinhead:1X03
- added MAIN_AUDIO: (no value), pinhead:1X03
- GENERAL_XPN: device pinhead:2X05 -> pinhead:2X13
- moved SCR 48.3 mm to (25.0, 4.70), turned to 0 degrees
- moved KNOBBOARD 43.2 mm to (54.6, 5.08), turned to 0 degrees
- moved PORTBOARD 34.7 mm to (71.1, 19.1), turned to 90 degrees
- moved BUTTONS 12.7 mm to (7.62, 33.0)
- renumbered U$1 to TEENSY_3.6
Connections:
- new net AUDIO_0: GENERAL_XPN.11
- new net AUDIO_1: GENERAL_XPN.13
- new net AUDIO_2: GENERAL_XPN.15
- new net AUDIO_3: GENERAL_XPN.17
- new net AUDIO_4: GENERAL_XPN.19
- new net AUDIO_5: GENERAL_XPN.21
- new net AUDIO_6: GENERAL_XPN.23
- new net AUDIO_7: GENERAL_XPN.25
- new net TEENSY_L: GENERAL_XPN.7, TEENSY_3.6.21/DAC0
- new net TEENSY_R: GENERAL_XPN.9, TEENSY_3.6.A22/DAC1
- new net XPN_CV0: GENERAL_XPN.12
- new net XPN_CV1: GENERAL_XPN.14
- new net XPN_CV2: GENERAL_XPN.16
- new net XPN_CV3: GENERAL_XPN.18
- new net XPN_CV4: GENERAL_XPN.20
- new net XPN_CV5: GENERAL_XPN.22
- new net XPN_CV6: GENERAL_XPN.24
- new net XPN_CV7: GENERAL_XPN.26
- net AGND: now also MAIN_AUDIO.3; no longer AUDIO_MAIN.2
- net AUDIO_L: now also MAIN_AUDIO.1; no longer AUDIO_MAIN.1, GENERAL_XPN.7, TEENSY_3.6.21/DAC0
- net AUDIO_R: now also MAIN_AUDIO.2; no longer AUDIO_MAIN.3, GENERAL_XPN.9, TEENSY_3.6.A22/DAC1
Routing:
- net AUDIO_L: track 76.9 -> 11.3 mm
- net ROTENC3_B: track 81.0 -> 21.4 mm
- net ROTENC4_A: track 79.0 -> 21.4 mm, vias 1 -> 0
- net MIDIIN1: track 27.0 -> 83.7 mm
- net AUDIO_R: track 65.8 -> 12.0 mm
- net MIDIOUT1: track 24.4 -> 75.5 mm
- net USBDATA+: track 32.8 -> 81.8 mm
- net MIDIIN2: track 9.72 -> 55.1 mm, vias 0 -> 1
- net ROTENC2_A: track 54.6 -> 10.1 mm, vias 1 -> 0
- net +5V: track 57.1 -> 101.4 mm, vias 1 -> 0
- net MIDIOUT2: track 10.1 -> 54.0 mm
- net USBDATA-: track 30.9 -> 73.2 mm
- net ROTENC1_B: track 50.6 -> 9.75 mm, vias 1 -> 0
- net SCR_DC: track 42.9 -> 4.59 mm, vias 2 -> 0
- net ROTENC4_B: track 58.1 -> 21.4 mm, vias 3 -> 0
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