File: Audio Mixer/audio_mixer.brd (EAGLE design)
At the start: 160 x 100 mm, 0 parts

Commit message: Audio Mixer half done
Parts:
- added C1, C2, C22, C23, C24, C25, C3, C31, C33, C34, C35, C4, C5, C6, C7, C8: 0.1u, rcl:C025-030X050
- added C10, C11, C12, C9: 10u, rcl:E5-10,5
- added C13, C14: 15n, rcl:C025-030X050
- added C15: 100u, rcl:E5-10,5
- added C16, C19, C20, C21: 2.2u, rcl:E2,5-6
- added C17, C18: 56n, rcl:C025-030X050
- added C26, C27, C28, C29: 47n, rcl:C025-030X050
- added C30, C32: 1000u, rcl:C050-050X075
- added IC1: LM747H, linear:H10C
- added R1, R10, R11, R12, R13, R14, R15, R16, R17, R18, R19, R2, R20, R3, R4, R5, R6, R7, R8, R9: (no value), rcl:R0805
- added R21, R22, R23, R24, R25, R26, R27, R28, R29, R30: (no value), rcl:PT-10
- added U1: TDA1524A, TDA1524A:DIP762W46P254L2160H470Q18P
Connections:
- new net +12V: C11.+, IC1.2, IC1.8
- new net -12V: C10.-, C9.-, IC1.5
- new net AGND: C11.-, C9.+
- new net GND: U1.18
- new net N$1: C1.1, R1.1
- new net N$10: R1.2, R21.3
- new net N$11: R2.2, R22.3
- new net N$12: R23.3, R3.2
- new net N$13: R24.3, R4.2
- new net N$14: R25.3, R5.2
- new net N$15: R26.3, R6.2
- new net N$16: R27.3, R7.2
- new net N$17: R28.3, R8.2
- new net N$18: C12.+, R10.1, R9.1
- new net N$19: IC1.1, R10.2, R29.3
- new net N$2: C10.+, IC1.4, IC1.6, R21.2, R22.2, R23.2, R24.2, R25.2, R26.2, R27.2, R28.2
- new net N$20: IC1.3, R21.1, R22.1, R23.1, R24.1, R29.1
- new net N$21: IC1.7, R25.1, R26.1, R27.1, R28.1, R30.2
- new net N$22: IC1.9, R30.3, R9.2
- new net N$23: C12.-, U1.15, U1.4
- new net N$3: C2.1, R2.1
- new net N$4: C3.1, R3.1
- new net N$5: C4.1, R4.1
- new net N$6: C5.1, R5.1
- new net N$7: C6.1, R6.1
- new net N$8: C7.1, R7.1
- new net N$9: C8.1, R8.1
- new net VP: U1.3

Commit message: mixer schematic functionally done, todo labels and brd
Parts:
- removed C13, C14: 15n, rcl:C025-030X050
- removed C15: 100u, rcl:E5-10,5
- removed C16, C19, C20, C21: 2.2u, rcl:E2,5-6
- removed C17, C18: 56n, rcl:C025-030X050
- removed C22, C23, C24, C25, C31, C33, C34, C35: 0.1u, rcl:C025-030X050
- removed C26, C27, C28, C29: 47n, rcl:C025-030X050
- removed C30, C32: 1000u, rcl:C050-050X075
- removed IC1: LM747H, linear:H10C
- removed R11, R12, R13, R14, R15, R16, R17, R18, R19, R20: (no value), rcl:R0805
- removed R21, R22, R23, R24, R25, R26, R27, R28, R29, R30: (no value), rcl:PT-10
- removed U1: TDA1524A, TDA1524A:DIP762W46P254L2160H470Q18P
- added IC2: LM747CN, linear:DIL14
- added VR1: 10k, rcl:PT-10
- added VR10, VR2, VR3, VR4, VR5, VR6, VR7, VR8, VR9: (no value), rcl:PT-10
- R1, R2, R3, R4, R5, R6, R7, R8: value (none) -> 1k
- R10, R9: value (none) -> 10k
- moved C1 214.0 mm to (3.81, -114.3), turned to 0 degrees
- moved C4 199.8 mm to (3.81, -137.2), turned to 0 degrees
- moved C3 185.6 mm to (3.81, -129.5), turned to 0 degrees
- moved C2 171.6 mm to (3.81, -121.9), turned to 0 degrees
- moved R4 168.6 mm to (2.54, -109.2), turned to 0 degrees
- moved R3 159.3 mm to (2.54, -104.1), turned to 0 degrees
- moved R2 150.0 mm to (2.54, -99.1), turned to 0 degrees
- moved R1 140.9 mm to (2.54, -94.0), turned to 0 degrees
- moved R10 127.3 mm to (2.54, -66.0), turned to 0 degrees
- moved R9 119.6 mm to (2.54, -61.0), turned to 0 degrees
- moved C12 49.1 mm to (6.35, -6.35), turned to 0 degrees
Connections:
- removed net GND: U1.18
- removed net N$2 (its old number): C10.+, IC1.4, IC1.6, R21.2, R22.2, R23.2, R24.2, R25.2, R26.2, R27.2, R28.2
- removed net N$20: IC1.3, R21.1, R22.1, R23.1, R24.1, R29.1
- removed net N$23: C12.-, U1.15, U1.4
- removed net VP: U1.3
- new net INPUT1: C1.2
- new net INPUT2: C2.2
- new net INPUT3: C3.2
- new net INPUT4: C4.2
- new net INPUT5: C5.2
- new net INPUT6: C6.2
- new net INPUT7: C7.2
- new net INPUT8: C8.2
- new net N$18: R2.2, VR2.2
- new net OUTPUT: C12.-
- net +12V: now also IC2.13, IC2.9; no longer IC1.2, IC1.8
- net -12V: now also IC2.4; no longer IC1.5
- net AGND: now also C10.+, IC2.2, IC2.6, VR1.1, VR10.1, VR2.1, VR3.1, VR4.1, VR5.1, VR6.1, VR7.1, VR8.1, VR9.2
- net N$10: now also R3.2, VR3.2; no longer R1.2, R21.3
- net N$11: now also IC2.7, VR5.3, VR6.3, VR7.3, VR8.3, VR9.3; no longer R2.2, R22.3
- net N$12: now also IC2.1, VR1.3, VR10.3, VR2.3, VR3.3, VR4.3; no longer R23.3, R3.2
- net N$13: now also R1.2, VR1.2; no longer R24.3, R4.2
- net N$14: now also R4.2, VR4.2; no longer R25.3, R5.2
- net N$15: now also R5.2, VR5.2; no longer R26.3, R6.2
- net N$16: now also R6.2, VR6.2; no longer R27.3, R7.2
- net N$17: now also R7.2, VR7.2; no longer R28.3, R8.2
- net N$19: now also IC2.12, VR10.2; no longer IC1.1, R29.3
- net N$21: now also R8.2, VR8.2; no longer IC1.7, R25.1, R26.1, R27.1, R28.1, R30.2
- net N$22: now also IC2.10, VR9.1; no longer IC1.9, R30.3

Commit message: Mixer Design complete
Parts:
- removed IC2: LM747CN, linear:DIL14
- added C13: 10u, rcl:E5-10,5
- added C14, C15, C16, C17, C18, C19, C20, C21, C22, C24: 0.1u, rcl:C025-030X050
- added IC1: OPA2134P, linear:DIL08
- added INPUT_AUDIO: (no value), pinhead:2X09
- added OUTPUT_AUDIO, POWER: (no value), pinhead:1X03
- added R11, R12, R13, R14, R15, R16, R17, R18, R19, R21: 1k, rcl:R0805
- added VR11, VR16: 10k, rcl:PT-10
- added VR12, VR13, VR14, VR15, VR17, VR18, VR19, VR21: (no value), rcl:PT-10
- VR6: value (none) -> 10k
- moved VR9 313.6 mm to (80.0, 78.7)
- moved VR10 302.2 mm to (92.7, 78.7)
- moved VR1 228.9 mm to (33.0, 77.5)
- moved VR4 228.9 mm to (33.0, 31.8)
- moved VR2 227.6 mm to (33.0, 61.0)
- moved VR3 227.6 mm to (33.0, 45.7)
- moved C1 194.6 mm to (14.0, 80.0)
- moved C2 194.6 mm to (14.0, 72.4)
- moved C3 194.6 mm to (14.0, 64.8)
- moved C4 194.6 mm to (14.0, 57.1)
- moved R1 167.5 mm to (21.6, 72.4)
- moved R2 167.5 mm to (21.6, 67.3)
- moved R3 167.5 mm to (21.6, 62.2)
- moved R4 167.5 mm to (21.6, 57.1)
- moved R10 158.9 mm to (88.9, 67.3), turned to 90 degrees
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Connections:
- removed net +12V: C11.+, IC2.13, IC2.9
- removed net -12V: C10.-, C9.-, IC2.4
- removed net INPUT1: C1.2
- removed net INPUT2: C2.2
- removed net INPUT3: C3.2
- removed net INPUT4: C4.2
- removed net INPUT5: C5.2
- removed net INPUT6: C6.2
- removed net INPUT7: C7.2
- removed net INPUT8: C8.2
- removed net OUTPUT: C12.-
- new net +15V: C11.+, IC1.8, POWER.1
- new net -15V: C10.-, C9.-, IC1.4, POWER.2
- new net L_INPUT1: C15.2, INPUT_AUDIO.1
- new net L_INPUT2: C16.2, INPUT_AUDIO.3
- new net L_INPUT3: C17.2, INPUT_AUDIO.5
- new net L_INPUT4: C18.2, INPUT_AUDIO.7
- new net L_INPUT5: C19.2, INPUT_AUDIO.9
- new net L_INPUT6: C20.2, INPUT_AUDIO.11
- new net L_INPUT7: C21.2, INPUT_AUDIO.13
- new net L_INPUT8: C22.2, INPUT_AUDIO.15
- new net N$20: C13.+, R9.1
- new net N$23: R13.2, VR7.2
- new net N$24: VR1.1, VR2.1, VR3.1, VR4.1
- new net N$28: R7.2, VR13.2
- new net N$29: R5.2, VR11.2
- new net N$30: R6.2, VR12.2
- new net N$32: R8.2, VR14.2
- new net N$34: VR11.1, VR12.1, VR13.1, VR14.1, VR15.1, VR5.1, VR6.1, VR7.1, VR8.1
- new net N$35: C18.1, R15.1
- new net N$36: R15.2, VR15.2
- new net N$37: IC1.6, VR15.3, VR16.3, VR17.3, VR18.3, VR19.3, VR21.3, VR6.3, VR7.3, VR8.3, VR9.3
- new net N$39: C19.1, R16.1
- new net N$40: C20.1, R17.1
- new net N$41: C21.1, R18.1
- new net N$42: R18.2, VR18.2
- new net N$43: R16.2, VR16.2
- new net N$44: R17.2, VR17.2
- new net N$45: C22.1, R19.1
- new net N$46: R19.2, VR19.2
- new net N$6: C14.1, R11.1
- new net N$7: R11.2, VR5.2
- new net N$8: C24.1, R21.1
- new net N$9: R21.2, VR21.2
- new net OUTPUT_L: C13.-, OUTPUT_AUDIO.1
- new net OUTPUT_R: C12.-, OUTPUT_AUDIO.2
- new net R_INPUT1: C1.2, INPUT_AUDIO.2
- new net R_INPUT2: C2.2, INPUT_AUDIO.4
- new net R_INPUT3: C3.2, INPUT_AUDIO.6
- new net R_INPUT4: C4.2, INPUT_AUDIO.8
- new net R_INPUT5: C5.2, INPUT_AUDIO.10
- new net R_INPUT6: C6.2, INPUT_AUDIO.12
- new net R_INPUT7: C7.2, INPUT_AUDIO.14
- new net R_INPUT8: C8.2, INPUT_AUDIO.16
- new net TEENSY_L: C24.2, INPUT_AUDIO.17
- new net TEENSY_R: C14.2, INPUT_AUDIO.18
- net AGND: now also IC1.3, IC1.5, OUTPUT_AUDIO.3, POWER.3, VR16.1, VR17.1, VR18.1, VR19.1; no longer IC2.2, IC2.6, VR1.1, VR2.1, VR3.1, VR4.1, VR5.1, VR6.1, VR7.1, VR8.1
- net N$11: now also C15.1, R12.1; no longer IC2.7, VR5.3, VR6.3, VR7.3, VR8.3, VR9.3
- net N$12: now also IC1.2, VR11.3, VR12.3, VR13.3, VR14.3, VR5.3; no longer IC2.1
- net N$15: now also C16.1, R13.1; no longer R5.2, VR5.2
- net N$16: now also C17.1, R14.1; no longer R6.2, VR6.2
- net N$17: now also R14.2, VR8.2; no longer R7.2, VR7.2
- net N$19: now also IC1.1; no longer IC2.12
- net N$2: no longer R9.1
- net N$21: now also R12.2, VR6.2; no longer R8.2, VR8.2
- net N$22: now also IC1.7; no longer IC2.10
Other:
- board size 160 x 100 mm -> 104.1 x 100 mm

Commit message: audio mixer comlpete!
Parts:
- removed C24: 0.1u, rcl:C025-030X050
- removed R21: 1k, rcl:R0805
- removed VR21: (no value), rcl:PT-10
- added C23: 10u, rcl:E5-10,5
- added R20: 10k, rcl:R0805
- added VR20: EVUF2A, pot:EVUF
- C10, C11, C12, C13, C9: value 10u -> 0.1u; device rcl:E5-10,5 -> rcl:C025-030X050
- C19, C20, C21, C22: value 0.1u -> 10u; device rcl:C025-030X050 -> rcl:E5-10,5
- R10, R9: value 10k -> 1k
- R19: value 1k -> 10k
- VR1, VR11, VR16, VR6: value 10k -> EVUF2A; device rcl:PT-10 -> pot:EVUF
- VR10, VR12, VR13, VR14, VR15, VR17, VR18, VR19, VR2, VR3, VR4, VR5, VR7, VR8, VR9: value (none) -> EVUF2A; device rcl:PT-10 -> pot:EVUF
- moved INPUT_AUDIO 273.2 mm to (66.0, 85.1)
- moved POWER 225.9 mm to (124.5, 16.5), turned to 90 degrees
- moved OUTPUT_AUDIO 205.8 mm to (11.4, 16.5), turned to 270 degrees
- moved R12 203.5 mm to (39.4, 72.4), turned to 180 degrees
- moved R15 192.8 mm to (39.4, 50.8), turned to 180 degrees
- moved VR6 186.9 mm to (118.1, 61.0)
- moved C20 184.1 mm to (114.3, 16.5), turned to 90 degrees
- moved R13 183.0 mm to (11.4, 50.8), turned to 180 degrees
- moved R14 182.2 mm to (25.4, 50.8), turned to 180 degrees
- moved C21 173.4 mm to (101.6, 16.5), turned to 90 degrees
- moved VR15 169.6 mm to (39.4, 61.0)
- moved C15 168.9 mm to (44.5, 50.8)
- moved R18 168.6 mm to (39.4, 29.2), turned to 180 degrees
- moved R17 167.9 mm to (25.4, 29.2), turned to 180 degrees
- moved R16 167.7 mm to (11.4, 29.2), turned to 180 degrees
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Connections:
- removed net N$12: IC1.2, VR1.3, VR10.3, VR11.3, VR12.3, VR13.3, VR14.3, VR2.3, VR3.3, VR4.3, VR5.3
- removed net N$19: IC1.1, R10.2, VR10.2
- removed net N$22: IC1.7, R9.2, VR9.1
- removed net N$24: VR1.1, VR2.1, VR3.1, VR4.1
- removed net N$34: VR11.1, VR12.1, VR13.1, VR14.1, VR15.1, VR5.1, VR6.1, VR7.1, VR8.1
- removed net N$37: IC1.6, VR15.3, VR16.3, VR17.3, VR18.3, VR19.3, VR21.3, VR6.3, VR7.3, VR8.3, VR9.3
- new net LEFT_OP_OUT: IC1.7, R20.2, VR20.1
- new net L_OP_IN: IC1.6, VR10.2, VR11.2, VR12.2, VR13.2, VR14.2, VR15.2, VR16.2, VR17.2, VR18.2, VR20.2
- new net RIGHT_OP_OUT: IC1.1, R19.2, VR19.1
- new net R_OP_IN: IC1.2, VR1.2, VR19.2, VR2.2, VR3.2, VR4.2, VR5.2, VR6.2, VR7.2, VR8.2, VR9.2
- net +15V: now also C20.+; no longer C11.+
- net -15V: now also C19.-, C21.-; no longer C10.-, C9.-
- net AGND: now also C19.+, C20.-, C21.+, VR1.3, VR10.3, VR11.3, VR12.3, VR13.3, VR14.3, VR15.3, VR16.3, VR17.3, VR18.3, VR19.3, VR2.3, VR20.3, VR3.3, VR4.3, VR5.3, VR6.3, VR7.3, VR8.3, VR9.3; no longer C10.+, C11.-, C9.+, VR10.1, VR16.1, VR17.1, VR18.1, VR19.1, VR9.2
- net L_INPUT1: now also C10.2; no longer C15.2
- net L_INPUT2: now also C11.2; no longer C16.2
- net L_INPUT3: now also C12.2; no longer C17.2
- net L_INPUT4: now also C13.2; no longer C18.2
- net L_INPUT5: now also C14.2; no longer C19.2
- net L_INPUT6: now also C15.2; no longer C20.2
- net L_INPUT7: now also C16.2; no longer C21.2
- net L_INPUT8: now also C17.2; no longer C22.2
- net N$10: now also VR3.1; no longer VR3.2
- net N$11: now also C11.1, R11.1; no longer C15.1, R12.1
- net N$13: now also VR1.1; no longer VR1.2
- net N$14: now also VR4.1; no longer VR4.2
- net N$15: now also C12.1, R12.1; no longer C16.1, R13.1
- net N$16: now also C13.1, R13.1; no longer C17.1, R14.1
- net N$17: now also R13.2, VR13.1; no longer R14.2, VR8.2
- net N$18: now also VR2.1; no longer VR2.2
- net N$2: now also C22.+, R19.1; no longer C12.+, R10.1
- net N$20: now also C23.+, R20.1; no longer C13.+, R9.1
- net N$21: now also R11.2, VR11.1; no longer R12.2, VR6.2
- net N$23: now also R12.2, VR12.1; no longer R13.2, VR7.2
- net N$28: now also VR7.1; no longer VR13.2
- net N$29: now also VR5.1; no longer VR11.2
- net N$30: now also VR6.1; no longer VR12.2
- net N$32: now also VR8.1; no longer VR14.2
- net N$35: now also C14.1, R14.1; no longer C18.1, R15.1
- net N$36: now also R14.2, VR14.1; no longer R15.2, VR15.2
- net N$39: now also C15.1, R15.1; no longer C19.1, R16.1
- net N$40: now also C16.1, R16.1; no longer C20.1, R17.1
- net N$41: now also C17.1, R17.1; no longer C21.1, R18.1
- net N$42: now also R17.2, VR17.1; no longer R18.2, VR18.2
- net N$43: now also R15.2, VR15.1; no longer R16.2, VR16.2
- net N$44: now also R16.2, VR16.1; no longer R17.2, VR17.2
- net N$45: now also C18.1, R18.1; no longer C22.1, R19.1
- net N$46: now also R18.2, VR18.1; no longer R19.2, VR19.2
- net N$6: now also C9.1, R9.1; no longer C14.1, R11.1
- net N$7: now also R9.2, VR9.1; no longer R11.2, VR5.2
- net N$8: now also C10.1, R10.1; no longer C24.1, R21.1
- net N$9: now also R10.2, VR10.1; no longer R21.2, VR21.2
- net OUTPUT_L: now also C23.-; no longer C13.-
- net OUTPUT_R: now also C22.-; no longer C12.-
- net TEENSY_L: now also C18.2; no longer C24.2
- net TEENSY_R: now also C9.2; no longer C14.2
Routing:
- net R_OP_IN: track 0.00 -> 174.4 mm
- net L_OP_IN: track 0.00 -> 168.9 mm
- net TEENSY_R: track 0.00 -> 94.6 mm
- net R_INPUT8: track 0.00 -> 84.2 mm
- net R_INPUT6: track 0.00 -> 84.1 mm
- net L_INPUT7: track 0.00 -> 83.5 mm
- net R_INPUT5: track 0.00 -> 73.9 mm
- net R_INPUT3: track 0.00 -> 73.2 mm
- net L_INPUT8: track 0.00 -> 73.0 mm
- net R_INPUT7: track 0.00 -> 72.9 mm
- net TEENSY_L: track 0.00 -> 69.3 mm
- net +15V: track 0.00 -> 65.4 mm
- net R_INPUT2: track 0.00 -> 63.0 mm
- net R_INPUT4: track 0.00 -> 62.6 mm
- net L_INPUT4: track 0.00 -> 60.1 mm
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- added copper zone on layer 1, net AGND
Other:
- board size 104.1 x 100 mm -> 132.1 x 101.3 mm
- board text added: "1 2 3 4 5 6 7 8 T"
- board text added: "9 Channel Stereo Audio Mixer"
- board text added: "L Gain Adj"
- board text added: "Left Level Control"
- board text added: "R Gain Adj"
- board text added: "R L"
- board text added: "Right Level Control"

Commit message: old seperate files
Parts:
- VR1, VR10, VR11, VR12, VR13, VR14, VR15, VR16, VR17, VR18, VR2, VR3, VR4, VR5, VR6, VR7, VR8, VR9: value EVUF2A -> (none); device pot:EVUF -> rcl:RTRIM3339P
- moved VR13 5.39 mm to (10.2, 57.1)
- moved VR15 5.24 mm to (40.6, 55.9)
- moved VR2 5.24 mm to (100.3, 81.3)
- moved VR14 4.58 mm to (29.2, 57.1)
- moved VR17 4.58 mm to (29.2, 35.6)
- moved VR18 4.58 mm to (41.9, 35.6)
- moved VR7 4.58 mm to (88.9, 36.8)
- moved VR11 3.59 mm to (29.2, 85.1)
- moved VR1 3.59 mm to (90.2, 80.0), turned to 90 degrees
- moved VR16 2.84 mm to (12.7, 36.8)
- moved VR4 2.84 mm to (90.2, 59.7)
- moved VR10 2.54 mm to (11.4, 82.5)
- moved VR12 2.54 mm to (41.9, 82.5)
- moved VR3 1.80 mm to (116.8, 81.3)
- moved VR5 1.80 mm to (104.1, 62.2)
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Routing:
- net R_OP_IN: track 174.4 -> 18.5 mm
- net L_OP_IN: track 168.9 -> 15.1 mm
- net N$14: track 0.00 -> 6.26 mm
- net N$28: track 0.00 -> 6.26 mm
- net N$13: track 0.00 -> 6.26 mm
- net N$30: track 0.00 -> 6.26 mm
- net N$29: track 0.00 -> 6.26 mm
- net N$7: track 0.00 -> 6.26 mm
- net N$32: track 0.00 -> 6.26 mm
- net N$18: track 0.00 -> 6.26 mm
- net N$10: track 0.00 -> 6.26 mm
- net N$36: track 3.28 -> 0.40 mm
- net N$42: track 3.28 -> 0.40 mm
- net N$6: track 0.00 -> 2.86 mm
- net N$5: track 0.00 -> 2.86 mm
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