File: Main Board/main.sch (EAGLE design)
At the start: 7 parts

Commit message: Main Board Complete!
Parts:
- added SDPIN1, SDPIN2, SDPIN3, SDPIN4, SDPIN5, SDPIN6, SDPIN7, SDPIN8: (no value), wirepad:1,6/0,8
- GENERAL_XPN: device pinhead:PINHD-2X13 -> pinhead:PINHD-2X11
Connections:
- net AUDIO_L renamed OUTPUT_L
- net AUDIO_R renamed OUTPUT_R
- net SPI_CLK renamed XPN_CLK
- net SPI_MISO renamed XPN_MISO
- net SPI_MOSI renamed XPN_MOSI
- removed net AUDIO_0: GENERAL_XPN.11
- removed net AUDIO_1: GENERAL_XPN.13
- removed net AUDIO_2: GENERAL_XPN.15
- removed net AUDIO_3: GENERAL_XPN.17
- removed net AUDIO_4: GENERAL_XPN.19
- removed net AUDIO_5: GENERAL_XPN.21
- removed net AUDIO_6: GENERAL_XPN.23
- removed net AUDIO_7: GENERAL_XPN.25
- removed net N$10: TEENSY_3.6.25
- removed net N$11: TEENSY_3.6.26
- removed net N$12: TEENSY_3.6.27
- removed net N$25: TEENSY_3.6.15/A1
- removed net N$26: TEENSY_3.6.14/A0
- removed net N$6: TEENSY_3.6.6
- removed net N$9: TEENSY_3.6.24
- removed net SPI_CS: GENERAL_XPN.8
- removed net XPN_CV0: GENERAL_XPN.12
- removed net XPN_CV1: GENERAL_XPN.14
- removed net XPN_CV2: GENERAL_XPN.16
- removed net XPN_CV3: GENERAL_XPN.18
- removed net XPN_CV4: GENERAL_XPN.20
- removed net XPN_CV5: GENERAL_XPN.22
- removed net XPN_CV6: GENERAL_XPN.24
- removed net XPN_CV7: GENERAL_XPN.26
- new net XPN_CS0: GENERAL_XPN.8, TEENSY_3.6.6
- new net XPN_CS1: GENERAL_XPN.10, TEENSY_3.6.24
- new net XPN_CS2: GENERAL_XPN.12, TEENSY_3.6.25
- new net XPN_CS3: GENERAL_XPN.14, TEENSY_3.6.26
- new net XPN_CS4: GENERAL_XPN.16, TEENSY_3.6.27
- new net XPN_CS5: GENERAL_XPN.18, TEENSY_3.6.15/A1
- new net XPN_CS6: GENERAL_XPN.20, TEENSY_3.6.14/A0
- new net XPN_CS7: GENERAL_XPN.22, TEENSY_3.6.A10
- net +5V: now also SDPIN4.P
- net GND: now also SDPIN6.P
- net SDCLK: now also SDPIN5.P
- net SDCMD: now also SDPIN3.P
- net SDDATA0: now also SDPIN7.P
- net SDDATA1: now also SDPIN8.P
- net SDDATA2: now also SDPIN1.P
- net SDDATA3: now also SDPIN2.P
- net TEENSY_L: now also GENERAL_XPN.9; no longer GENERAL_XPN.7
- net TEENSY_R: now also GENERAL_XPN.7; no longer GENERAL_XPN.9
Other:
- note added: "Note: If I'm not mistaken all (Teensy) digital pins can be used as SPI chip select pins"
- note added: "Note: Other audio inputs go directly into mixer circuit (src of MAIN_AUDIO output)"
- note added: "ie. Output from mixer circuit"
- moved on the sheet: BUTTONS, KNOBBOARD, MAIN_AUDIO, PORTBOARD

Commit message: old seperate files
Parts:
- removed GENERAL_XPN: (no value), pinhead:PINHD-2X11
- removed MAIN_AUDIO: (no value), pinhead:PINHD-1X3
- added JP1, JP2, JP3, JP4, JP5, JP6, JP7, JP8: (no value), pinhead:PINHD-1X11
Connections:
- new net -12V: JP1.2, JP2.2, JP3.2, JP4.2, JP5.2, JP6.2, JP7.2, JP8.2
- new net L_INPUT1: JP1.7, JP2.7, JP3.7, JP4.7, JP5.7, JP6.7, JP7.7, JP8.7
- new net R_INPUT1: JP1.6, JP2.6, JP3.6, JP4.6, JP5.6, JP6.6, JP7.6, JP8.6
- net +12V: now also JP1.1, JP2.1, JP3.1, JP4.1, JP5.1, JP6.1, JP7.1, JP8.1; no longer GENERAL_XPN.3
- net +3V3: now also SDPIN4.P
- net +5V: now also JP1.3, JP2.3, JP3.3, JP4.3, JP5.3, JP6.3, JP7.3, JP8.3; no longer GENERAL_XPN.1, SDPIN4.P
- net AGND: now also JP1.5, JP2.5, JP3.5, JP4.5, JP5.5, JP6.5, JP7.5, JP8.5; no longer MAIN_AUDIO.3
- net GND: now also JP1.4, JP2.4, JP3.4, JP4.4, JP5.4, JP6.4, JP7.4, JP8.4; no longer GENERAL_XPN.5
- net JOYSTICK_Y: now also TEENSY_3.6.A10; no longer TEENSY_3.6.22/A8
- net OUTPUT_L: no longer MAIN_AUDIO.1
- net OUTPUT_R: no longer MAIN_AUDIO.2
- net TEENSY_L: no longer GENERAL_XPN.9
- net TEENSY_R: no longer GENERAL_XPN.7
- net XPN_CLK: now also JP1.11, JP2.11, JP3.11, JP4.11, JP5.11, JP6.11, JP7.11, JP8.11; no longer GENERAL_XPN.2
- net XPN_CS0: now also JP1.8; no longer GENERAL_XPN.8
- net XPN_CS1: now also JP2.8; no longer GENERAL_XPN.10
- net XPN_CS2: now also JP3.8; no longer GENERAL_XPN.12
- net XPN_CS3: now also JP4.8; no longer GENERAL_XPN.14
- net XPN_CS4: now also JP5.8; no longer GENERAL_XPN.16
- net XPN_CS5: now also JP6.8; no longer GENERAL_XPN.18
- net XPN_CS6: now also JP7.8; no longer GENERAL_XPN.20
- net XPN_CS7: now also JP8.8, TEENSY_3.6.22/A8; no longer GENERAL_XPN.22, TEENSY_3.6.A10
- net XPN_MISO: now also JP1.9, JP2.9, JP3.9, JP4.9, JP5.9, JP6.9, JP7.9, JP8.9; no longer GENERAL_XPN.6
- net XPN_MOSI: now also JP1.10, JP2.10, JP3.10, JP4.10, JP5.10, JP6.10, JP7.10, JP8.10; no longer GENERAL_XPN.4
Other:
- note removed: "Note: Other audio inputs go directly into mixer circuit (src of MAIN_AUDIO output)"
- note removed: "ie. Output from mixer circuit"
- moved on the sheet: BUTTONS, KNOBBOARD, PORTBOARD, SCR-1, SCR-10, SCR-11, SCR-12, SCR-13, SCR-14, SCR-15, SCR-16, SCR-17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
